File: brelok_ext.brd (EAGLE design)
At the start: 100 x 80 mm, 18 parts, among them IC1 STM32F103C8T, IC2 AT24CP, M1 WIRELESS-NRF24L01

Commit message: Updated
Parts:
- removed IC2: AT24CP, atmel:DIL08
- added IC3: 24C01SN, microchip:SO-08
- added X1: SPARKFUN_USB-MICROB, antduino:SPARKFUN_USB-MICROB
- moved SL1 8.67 mm to (17.1, 54.7), turned to 90 degrees
- moved R1 2.20 mm to (12.6, 56.8)
- moved RESET 1.93 mm to (7.06, 57.4)
- moved R3 0.68 mm to (39.0, 76.2), turned to 270 degrees
- moved IC1 0.06 mm to (26.2, 64.3)
Connections:
- net GND: now also IC3.1, IC3.2, IC3.3, IC3.4, IC3.7, X1.GND
- net N$21: now also IC3.6; no longer IC2.6
- net N$22: now also IC3.5; no longer IC2.5
- net N$23: now also IC1.32, X1.D-; no longer IC2.4
- net N$24: now also IC1.33, X1.D+; no longer IC2.1, IC2.2, IC2.3, IC2.7
- net VCC: now also IC3.8; no longer IC2.8
Routing:
- net GND: track 162.0 -> 190.1 mm
- net N$10: track 5.75 -> 13.7 mm
- net N$21: track 0.00 -> 7.49 mm
- net VCC: track 81.8 -> 89.3 mm
- net N$12: track 5.01 -> 11.6 mm
- net N$22: track 0.00 -> 6.05 mm
- net N$9: track 53.7 -> 59.5 mm
- net N$19: track 43.8 -> 48.6 mm
- net N$24: track 0.00 -> 3.72 mm
- net N$23: track 0.00 -> 3.65 mm
- net N$20: track 8.26 -> 5.39 mm, vias 3 -> 5
- net N$2: track 27.4 -> 30.0 mm
- net N$8: track 27.9 -> 30.1 mm
- net N$18: track 50.9 -> 51.5 mm

Commit message: Made working prototype
Parts:
- added U$2: CR2025_SMD, CR2025:SMD
- moved R5 12.8 mm to (37.6, 71.9)
- moved R4 10.7 mm to (37.6, 69.8)
- moved M1 6.47 mm to (25.9, 63.6), flipped to the top, turned to 0 degrees
- moved LED1 4.58 mm to (48.8, 68.3)
- moved LED2 4.57 mm to (48.8, 63.5)
- moved R1 3.81 mm to (15.6, 59.1), turned to 180 degrees
- moved R2 3.57 mm to (3.81, 72.6)
- moved IC3 2.55 mm to (36.9, 61.6)
- moved RESET 1.52 mm to (8.59, 57.4)
- moved BOOT 1.44 mm to (8.64, 73.9)
- moved C2 1.27 mm to (24.0, 72.4), turned to 0 degrees
- moved C1 1.14 mm to (29.7, 72.4), turned to 180 degrees
- moved SL1 0.51 mm to (17.1, 54.2), turned to 180 degrees
Connections:
- net GND: now also U$2.-
- net VCC: now also U$2.+
Routing:
- net N$34: track 0.00 -> 165.6 mm
- net GND: track 190.1 -> 167.1 mm, vias 0 -> 4
- net N$1: track 24.4 -> 7.30 mm
- net N$2: track 30.0 -> 13.6 mm
- net N$14: track 5.09 -> 21.2 mm
- net N$19: track 48.6 -> 64.6 mm, vias 2 -> 0
- net N$8: track 30.1 -> 43.7 mm, vias 2 -> 3
- net N$16: track 20.5 -> 9.35 mm
- net N$15: track 22.1 -> 11.5 mm
- net N$17: track 175.3 -> 165.6 mm
- net N$3: track 18.8 -> 10.1 mm, vias 0 -> 2
- net N$13: track 4.56 -> 10.2 mm
- net N$20: track 5.39 -> 0.00 mm, vias 5 -> 0
- net N$5: track 12.0 -> 7.22 mm, vias 0 -> 2
- net N$26: track 0.00 -> 4.57 mm
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- added copper zone on layer 1, net N$32
- added copper zone on layer 16, net N$33
Other:
- board size 100 x 80 mm -> 100.3 x 80 mm
